Commit message: changed robot design

File: urdf/gazebo_control.xacro (robot description, xacro)
@@ -5,6 +5,6 @@
          <right_joint>right_wheel_joint</right_joint>
          <left_joint>left_wheel_joint</left_joint>
-         <wheel_separation>0.35</wheel_separation>
-         <wheel_diameter>0.1</wheel_diameter>
+         <wheel_separation>0.66</wheel_separation>
+         <wheel_diameter>0.346</wheel_diameter>
          <max_linear_acceleration>10</max_linear_acceleration>
          <topic>cmd_vel</topic>

File: urdf/robot_core.xacro (robot description, xacro)
@@ -1,4 +1,4 @@
 <?xml version="1.0"?>
-<robot xmlns:xacro="http://www.ros.org/wiki/xacro" >
+<robot xmlns:xacro="http://www.ros.org/wiki/xacro">
       <xacro:include filename="inertial_macros.xacro" />
       <!-- Base link -->
@@ -15,8 +15,8 @@
             <origin xyz="0.15 0 0.075"/>
             <geometry>
-               <box size="0.3 0.3 0.15"/>
+               <box size="0.65 0.65 0.213"/>
             </geometry>
             <material name="chassis_material">
-               <color rgba="0.40 0.23 0.72 1.0"/>
+               <color rgba="0.573 0.239 0.254 1.0"/>
             </material>
          </visual>
@@ -24,8 +24,8 @@
             <origin xyz="0.15 0 0.075"/>
             <geometry>
-               <box size="0.3 0.3 0.15"/>
+               <box size="0.65 0.65 0.213"/>
             </geometry>
          </collision>
-         <xacro:inertial_box mass="0.5" x="0.3" y="0.3" z="0.15">
+         <xacro:inertial_box mass="0.9" x="0.65" y="0.65" z="0.213">
             <origin xyz="0.15 0 0.075" rpy="0 0 0"/>
          </xacro:inertial_box>
@@ -35,5 +35,5 @@
         <parent link="base_link"/>
         <child link="left_wheel"/>
-        <origin xyz="0 0.175 0" rpy="-${pi/2} 0 0"/>
+        <origin xyz="-0.1 0.353 0.048" rpy="-${pi/2} 0 0"/>
         <axis xyz="0 0 1"/>
       </joint>
@@ -41,16 +41,16 @@
          <visual>
             <geometry>
-               <cylinder radius="0.05" length="0.04"/>
+               <cylinder radius="0.173" length="0.04"/>
             </geometry>
             <material name="wheel_material">
-               <color rgba="0.0 0.0 0.0 1.0"/>
+               <color rgba="0.239 0.239 0.239 1.0"/>
             </material>
          </visual>
          <collision>
             <geometry>
-               <cylinder radius="0.05" length="0.04"/>
+               <cylinder radius="0.173" length="0.04"/>
             </geometry>
          </collision>
-         <xacro:inertial_cylinder mass="0.1" length="0.04" radius="0.05">
+         <xacro:inertial_cylinder mass="0.2" length="0.04" radius="0.173">
             <origin xyz="0 0 0" rpy="0 0 0"/>
          </xacro:inertial_cylinder>
@@ -60,5 +60,5 @@
         <parent link="base_link"/>
         <child link="right_wheel"/>
-        <origin xyz="0 -0.175 0" rpy="${pi/2} 0 0"/>
+        <origin xyz="-0.1 -0.353 0.048" rpy="${pi/2} 0 0"/>
         <axis xyz="0 0 -1"/>
       </joint>
@@ -66,16 +66,16 @@
          <visual>
             <geometry>
-               <cylinder radius="0.05" length="0.04"/>
+               <cylinder radius="0.173" length="0.04"/>
             </geometry>
             <material name="wheel_material">
-                <color rgba="0.0 0.0 0.0 1.0"/>
+                <color rgba="0.239 0.239 0.239 1.0"/>
             </material>
          </visual>
          <collision>
             <geometry>
-               <cylinder radius="0.05" length="0.04"/>
+               <cylinder radius="0.173" length="0.04"/>
             </geometry>
          </collision>
-            <xacro:inertial_cylinder mass="0.1" length="0.04" radius="0.05">
+            <xacro:inertial_cylinder mass="0.2" length="0.04" radius="0.173">
             <origin xyz="0 0 0" rpy="0 0 0"/>
          </xacro:inertial_cylinder>
@@ -85,10 +85,10 @@
         <parent link="chassis"/>
         <child link="castor_wheel"/>
-        <origin xyz="0.24 0 0"/>
+        <origin xyz="0.39 0 -0.048"/>
       </joint>
       <link name="castor_wheel">
          <visual>
             <geometry>
-               <sphere radius="0.05"/>
+               <sphere radius="0.08"/>
             </geometry>
             <material name="castor_material">
@@ -98,8 +98,8 @@
          <collision>
             <geometry>
-               <sphere radius="0.05"/>
+               <sphere radius="0.08"/>
             </geometry>
          </collision>
-         <xacro:inertial_sphere mass="0.1" radius="0.05">
+         <xacro:inertial_sphere mass="0.15" radius="0.08">
             <origin xyz="0 0 0" rpy="0 0 0"/>
          </xacro:inertial_sphere>
