Commit message: using gazebo control warehouse

File: urdf/lidar.xacro (robot description, xacro)
@@ -10,5 +10,5 @@
          <origin xyz="0 0 0"/>
          <geometry>
-            <cylinder length="0.04" radius="0.05"/>
+            <cylinder length="0.09" radius="0.1"/>
          </geometry>
          <material name="laser_material">

File: urdf/robot.urdf.xacro (robot description, xacro)
@@ -3,4 +3,7 @@
     <xacro:include filename="robot_core.xacro" />
     <xacro:include filename="gazebo_control.xacro" />
+    <!-- <xacro:include filename="ros2_control.xacro" /> -->
     <xacro:include filename="lidar.xacro" />
+    <!-- <xacro:include filename="camera.xacro" /> -->
+    <xacro:include filename="depth_camera.xacro" />
 </robot>

File: urdf/robot_core.xacro (robot description, xacro)
@@ -35,5 +35,5 @@
         <parent link="base_link"/>
         <child link="left_wheel"/>
-        <origin xyz="-0.1 0.353 0.048" rpy="-${pi/2} 0 0"/>
+        <origin xyz="0.2 0.353 0.048" rpy="-${pi/2} 0 0"/>
         <axis xyz="0 0 1"/>
       </joint>
@@ -60,5 +60,5 @@
         <parent link="base_link"/>
         <child link="right_wheel"/>
-        <origin xyz="-0.1 -0.353 0.048" rpy="${pi/2} 0 0"/>
+        <origin xyz="0.2 -0.353 0.048" rpy="${pi/2} 0 0"/>
         <axis xyz="0 0 -1"/>
       </joint>
@@ -85,5 +85,5 @@
         <parent link="chassis"/>
         <child link="castor_wheel"/>
-        <origin xyz="0.39 0 -0.048"/>
+        <origin xyz="-0.08 0 -0.048"/>
       </joint>
       <link name="castor_wheel">
